Commit message: Updated limited URDF, alignment of realsense, dataset splitting

File: urdfs/motoman_mh5_support_limited/urdf/mh5l_limited.urdf (robot description, URDF)
Before this commit: robot motoman_mh5l_limited, 10 links, 9 joints
Joints:
- joint joint_1_s: limit lower=0 upper=2.96705972839 effort=303.8 velocity=4.71238898038 -> lower=-0.78539816339 upper=1.57079632679 effort=303.8 velocity=4.71238898038
- joint joint_2_l: limit lower=-1.1344640138 upper=2.61799387799 effort=205.8 velocity=4.88692190558 -> lower=-0.994838 upper=1.57079632679 effort=205.8 velocity=4.88692190558
- joint joint_3_u: limit lower=-1.2217304764 upper=3.31612557879 effort=85.5 velocity=5.23598775598 -> lower=-0.872665 upper=2.44346 effort=85.5 velocity=5.23598775598
